File: mainboard/pcb/mainboard.kicad_pcb (KiCad board)
At the start: 4 copper layers, 205.3 x 78 mm, 201 parts, among them J1 B4B-XH-2(LF)(SN), J2 WAFER-SH1.0-3PWB, J3 AFC07-S50ECC-00, J4 WAFER-SH1.0-3PWB, J5 B4B-XH-2(LF)(SN), J8 B2B-XH-A(LF)(SN), J9 USB4105-GF-A-120, Q1 AON7264E, Q2 AON7264E, Q3 WSD40120DN56G, Q4 AON7264E, Q5 BSS138W, Q6 BSS138W, Q7 BSS138W, SW1 TS3425BA, SW2 TS3425BA, U1 TMC2209-LA, U10 TPS62933, U11 ST25R3916-AQW, U12 AP33772S, U13 TLV75733PDBV, U14 DRV8701E, U15 AL8861Y, U16 RP2350_80QFN, U17 TPS16630RGE, U2 TMC2209-LA, U5 LM74700, U6 W25Q128JVSS, U8 SN74LVC1G97DBVR, U9 PCA9306DC1, Y1 ABM8-272-T3, Y2 27.12MHz

Commit message: muscle: more TMC air
Changed lines of the file:
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@@
 		(sheetname "/")
 		(sheetfile "mainboard.kicad_sch")
-		(units
-			(unit
-				(name "A")
-				(pins "4" "5" "1" "2" "3")
-			)
-		)
 		(attr smd)
 		(duplicate_pad_numbers_are_jumpers no)
 		(fp_line
-			(start -3 -2.61)
-			(end 3 -2.61)
+			(start -3 -2.71)
+			(end 3 -2.71)
 			(stroke
 				(width 0.12)
@@
 		)
 		(fp_line
-			(start -3 2.61)
-			(end 3 2.61)
+			(start -3 2.71)
+			(end 3 2.71)
 			(stroke
 				(width 0.12)
@@
 		)
 		(fp_line
-			(start -3.7 2.8)
+			(start -3.7 2.9)
 			(end -3.7 -2.9)
 			(stroke
@@
 		(fp_line
 			(start 3.7 -2.9)
-			(end 3.7 2.8)
+			(end 3.7 2.9)
 			(stroke
 				(width 0.05)
@@
 		)
 		(fp_line
-			(start 3.7 2.8)
-			(end -3.7 2.8)
+			(start 3.7 2.9)
+			(end -3.7 2.9)
 			(stroke
 				(width 0.05)
@@
 			(pintype "passive")
 		)
+		(pad "5" smd rect
+			(at 0.806275 0.05 270)
+			(size 4.3 4.05)
+			(layers "B.Cu")
+			(net "VM")
+		)
 		(pad "5" thru_hole circle
 			(at 2.5 -1.8)
@@
 		)
 		(embedded_fonts no)
-		(model "${KICAD10_3DMODEL_DIR}/Package_DFN_QFN.3dshapes/DFN-8-1EP_6x5mm_Pitch1.27mm.step"
-			(offset
-				(xyz 0 0 0)
-			)
-			(scale
-				(xyz 1 1 1)
-			)
-			(rotate
-				(xyz 0 0 0)
-			)
-		)
 		(model "${KICAD10_3DMODEL_DIR}/Package_DFN_QFN.3dshapes/AO_DFN-8-1EP_5.55x5.2mm_P1.27mm_EP4.12x4.6mm.step"
 			(offset
 				(xyz 0 0 0)
-			)
-			(scale
-				(xyz 1 1 1)
-			)
-			(rotate
-				(xyz 0 0 0)
-			)
-		)
-		(model "${KICAD10_3DMODEL_DIR}/Package_DFN_QFN.3dshapes/DFN-8-1EP_6x5mm_P1.27mm_EP4x4mm.step"
-			(offset
-				(xyz 0 0 0)
